Commit message: Add files via upload
Controllers can now communicate with the hardware interface.

File: src/robot_description/urdf/robot_x/robot_x_macro.ros2_control.xacro (robot description, xacro)
@@ -26,5 +26,5 @@
         </xacro:unless>
       </hardware>
-      <joint name="${prefix}joint1">
+      <joint name="${prefix}linear_velocity_joint">
         <command_interface name="position">     <!-- Add/Remove interfaces as needed -->
           <param name="min">-1</param>
@@ -37,5 +37,5 @@
         <state_interface name="acceleration"/>
       </joint>
-      <joint name="${prefix}joint2">
+      <joint name="${prefix}angular_velocity_joint">
         <command_interface name="position">     <!-- Add/Remove interfaces as needed -->
           <param name="min">-1</param>
@@ -48,69 +48,4 @@
         <state_interface name="acceleration"/>
       </joint>
-      <joint name="${prefix}joint3">
-        <command_interface name="position">     <!-- Add/Remove interfaces as needed -->
-          <param name="min">-1</param>
-          <param name="max">1</param>
-        </command_interface>
-        <state_interface name="position">
-          <param name="initial_value">0.0</param>
-        </state_interface>
-        <state_interface name="velocity"/>
-        <state_interface name="acceleration"/>
-      </joint>
-      <joint name="${prefix}joint4">
-        <command_interface name="position">     <!-- Add/Remove interfaces as needed -->
-          <param name="min">-1</param>
-          <param name="max">1</param>
-        </command_interface>
-        <state_interface name="position">
-          <param name="initial_value">0.0</param>
-        </state_interface>
-        <state_interface name="velocity"/>
-        <state_interface name="acceleration"/>
-      </joint>
-      <joint name="${prefix}joint5">
-        <command_interface name="position">     <!-- Add/Remove interfaces as needed -->
-          <param name="min">-1</param>
-          <param name="max">1</param>
-        </command_interface>
-        <state_interface name="position">
-          <param name="initial_value">0.0</param>
-        </state_interface>
-        <state_interface name="velocity"/>
-        <state_interface name="acceleration"/>
-      </joint>
-      <joint name="${prefix}joint6">
-        <command_interface name="position">     <!-- Add/Remove interfaces as needed -->
-          <param name="min">-1</param>
-          <param name="max">1</param>
-        </command_interface>
-        <state_interface name="position">
-          <param name="initial_value">0.0</param>
-        </state_interface>
-        <state_interface name="velocity"/>
-        <state_interface name="acceleration"/>
-      </joint>
-      <sensor name="tcp_fts_sensor">            <!-- Remove/change sensors as needed -->
-        <state_interface name="fx"/>
-        <state_interface name="fy"/>
-        <state_interface name="fz"/>
-        <state_interface name="tx"/>
-        <state_interface name="ty"/>
-        <state_interface name="tz"/>
-        <param name="frame_id">tool0</param>    <!-- Change sensors as needed -->
-        <param name="min_fx">-100</param>
-        <param name="max_fx">100</param>
-        <param name="min_fy">-100</param>
-        <param name="max_fy">100</param>
-        <param name="min_fz">-200</param>
-        <param name="max_fz">200</param>
-        <param name="min_tx">-10</param>
-        <param name="max_tx">10</param>
-        <param name="min_ty">-10</param>
-        <param name="max_ty">10</param>
-        <param name="min_tz">-15</param>
-        <param name="max_tz">15</param>
-      </sensor>
     </ros2_control>
     <xacro:if value="$(arg sim_gazebo_classic)">

File: src/robot_description/urdf/robot_x/robot_x_macro.xacro (robot description, xacro)
@@ -4,9 +4,6 @@
   <xacro:include filename="$(find robot_description)/urdf/common/materials.xacro"/>
   <xacro:macro name="robot_x" params="prefix parent *origin">
-    <!-- LINKS -->
-    <!-- base link -->
     <link name="${prefix}base_link">
-      <!-- Default inertial for Gazebo - copy and edit block from 'common.xacro'
-           to get more realistic behavior -->
+      <!-- Add geometry or inertia properties -->
       <xacro:default_inertial/>
       <visual>
@@ -26,8 +23,7 @@
       </collision>
     </link>
-    <!-- link 1 -->
-    <link name="${prefix}link1">
+    <link name="${prefix}linear_velocity_link">
       <!-- Default inertial for Gazebo - copy and edit block from 'common.xacro'
-           to get more realistic behavior -->
+      to get more realistic behavior -->
       <xacro:default_inertial/>
       <visual>
@@ -48,6 +44,5 @@
       </collision>
     </link>
-    <!-- link 2 -->
-    <link name="${prefix}link2">
+    <link name="${prefix}angular_velocity_link">
       <!-- Default inertial for Gazebo - copy and edit block from 'common.xacro'
            to get more realistic behavior-->
@@ -69,100 +64,4 @@
       </collision>
     </link>
-    <!-- link 3 -->
-    <link name="${prefix}link3">
-      <!-- Default inertial for Gazebo - copy and edit block from 'common.xacro'
-           to get more realistic behavior-->
-      <xacro:default_inertial/>
-      <visual>
-        <origin xyz="0 0 0" rpy="0 0 0"/>
-        <geometry>
-          <cylinder length="0.2" radius="0.1"/>
-          <!--           <mesh filename="package://robot_description/meshes/robot_x/visual/link3.dae" /> -->
-        </geometry>
-        <material name="orange"/>
-      </visual>
-      <collision>
-        <origin xyz="0 0 0" rpy="0 0 0"/>
-        <geometry>
-          <cylinder length="0.2" radius="0.1"/>
-          <!--           <mesh filename="package://robot_description/meshes/robot_x/collision/link3.stl"  /> -->
-        </geometry>
-      </collision>
-    </link>
-    <!-- link 4 -->
-    <link name="${prefix}link4">
-      <!-- Default inertial for Gazebo - copy and edit block from 'common.xacro'
-           to get more realistic behavior-->
-      <xacro:default_inertial/>
-      <visual>
-        <origin xyz="0 0 0" rpy="0 0 0"/>
-        <geometry>
-          <cylinder length="0.1" radius="0.1"/>
-          <!--           <mesh filename="package://robot_description/meshes/robot_x/visual/link4.dae" /> -->
-        </geometry>
-        <material name="brown"/>
-      </visual>
-      <collision>
-        <origin xyz="0 0 0" rpy="0 0 0"/>
-        <geometry>
-          <cylinder length="0.1" radius="0.1"/>
-          <!--           <mesh filename="package://robot_description/meshes/robot_x/collision/link4.stl"  /> -->
-        </geometry>
-      </collision>
-    </link>
-    <!-- link 5 -->
-    <link name="${prefix}link5">
-      <!-- Default inertial for Gazebo - copy and edit block from 'common.xacro'
-           to get more realistic behavior-->
-      <xacro:default_inertial/>
-      <visual>
-        <origin xyz="0 0 0" rpy="0 0 0"/>
-        <geometry>
-          <cylinder length="0.15" radius="0.1"/>
-          <!--           <mesh filename="package://robot_description/meshes/robot_x/visual/link5.dae" /> -->
-        </geometry>
-        <material name="red"/>
-      </visual>
-      <collision>
-        <origin xyz="0 0 0" rpy="0 0 0"/>
-        <geometry>
-          <cylinder length="0.15" radius="0.1"/>
-          <!--           <mesh filename="package://robot_description/meshes/robot_x/collision/link5.stl" /> -->
-        </geometry>
-      </collision>
-    </link>
-    <!-- link 6 -->
-    <link name="${prefix}link6">
-      <!-- Default inertial for Gazebo - copy and edit block from 'common.xacro'
-           to get more realistic behavior-->
-      <xacro:default_inertial/>
-      <visual>
-        <origin xyz="0 0 0" rpy="0 0 0"/>
-        <geometry>
-          <cylinder length="0.05" radius="0.075"/>
-          <!--           <mesh filename="package://robot_description/meshes/robot_x/visual/link6.dae" /> -->
-        </geometry>
-        <material name="white"/>
-      </visual>
-      <collision>
-        <origin xyz="0 0 0" rpy="0 0 0"/>
-        <geometry>
-          <cylinder length="0.05" radius="0.075"/>
-          <!--           <mesh filename="package://robot_description/meshes/robot_x/collision/link6.stl" /> -->
-        </geometry>
-      </collision>
-    </link>
-    <!-- All-zero tool frame. This frame should correspond to the TOOL frame of the robot's controller.) -->
-    <link name="${prefix}tool0"/>
-    <!-- tool link -->
-    <!-- START Delete if not needed -->
-    <!-- Standard frames for industrial robots. Also useful for manipulators.
-         (ROS-I specs - https://wiki.ros.org/Industrial/Tutorials/WorkingWithRosIndustrialRobotSupportPackages#Standardised_links_.2F_frames)-->
-    <!-- This frame should correspond to the BASE coordinate system of robot's controller.) -->
-    <link name="${prefix}base"/>
-    <!-- Frame for mounting EEF models to a manipulator. x+ axis points forward (REP 103). -->
-    <link name="${prefix}flange"/>
-    <!-- END Delete if not needed  -->
-    <!-- END LINKS -->
     <!-- JOINTS -->
     <!-- base_joint fixes base_link to the environment -->
@@ -173,72 +72,19 @@
     </joint>
     <!-- joint 1 -->
-    <joint name="${prefix}joint1" type="revolute">
+    <joint name="${prefix}linear_velocity_joint" type="revolute">
       <origin xyz="0 0 0.3" rpy="${pi} 0 0"/>
-      <parent link="${prefix}base_link"/>
-      <child link="${prefix}link1"/>
       <axis xyz="0 0 1"/>
       <limit effort="0" lower="${radians(-180)}" upper="${radians(180)}" velocity="${radians(180)}"/>
+      <parent link="${prefix}base_link"/>  <!-- Specify parent link -->
+      <child link="${prefix}linear_velocity_link"/>  <!-- Specify child link -->
     </joint>
     <!-- joint 2 -->
-    <joint name="${prefix}joint2" type="revolute">
+    <joint name="${prefix}angular_velocity_joint" type="revolute">
       <origin xyz="0 0 -0.3" rpy="${pi/2} 0 0"/>
-      <parent link="${prefix}link1"/>
-      <child link="${prefix}link2"/>
       <axis xyz="0 0 1"/>
       <limit effort="0" lower="${radians(-180)}" upper="${radians(180)}" velocity="${radians(180)}"/>
+      <parent link="${prefix}linear_velocity_link"/>  <!-- Specify parent link -->
+      <child link="${prefix}angular_velocity_link"/>  <!-- Specify child link -->
     </joint>
-    <!-- joint 3 -->
-    <joint name="${prefix}joint3" type="revolute">
-      <origin xyz="0.8 0 0" rpy="0 0 0"/>
-      <parent link="${prefix}link2"/>
-      <child link="${prefix}link3"/>
-      <axis xyz="0 0 1"/>
-      <limit effort="0" lower="${radians(-90)}" upper="${radians(180)}" velocity="${radians(270)}"/>
-    </joint>
-    <!-- joint 4 -->
-    <joint name="${prefix}joint4" type="revolute">
-      <origin xyz="0.15 0 0" rpy="0 ${-pi/2} 0"/>
-      <parent link="${prefix}link3"/>
-      <child link="${prefix}link4"/>
-      <axis xyz="0 0 1"/>
-      <limit effort="0" lower="${radians(-360)}" upper="${radians(360)}" velocity="${radians(360)}"/>
-    </joint>
-    <!-- joint 5 -->
-    <joint name="${prefix}joint5" type="revolute">
-      <origin xyz="0 0 -0.15" rpy="0 ${pi/2} 0"/>
-      <parent link="${prefix}link4"/>
-      <child link="${prefix}link5"/>
-      <axis xyz="0 0 1"/>
-      <limit effort="0" lower="${radians(-120)}" upper="${radians(120)}" velocity="${radians(540)}"/>
-    </joint>
-    <!-- joint 6 -->
-    <joint name="${prefix}joint6" type="revolute">
-      <origin xyz="0.125 0 0" rpy="0 ${-pi/2} 0"/>
-      <parent link="${prefix}link5"/>
-      <child link="${prefix}link6"/>
-      <axis xyz="0 0 1"/>
-      <limit effort="0" lower="${radians(-360)}" upper="${radians(360)}" velocity="${radians(720)}"/>
-    </joint>
-    <!-- tool frame - fixed frame -->
-    <joint name="${prefix}joint6-tool0" type="fixed">
-      <parent link="${prefix}link6"/>
-      <child link="${prefix}tool0"/>
-      <origin xyz="0 0 -0.115" rpy="0 ${-pi} ${-pi/2}"/>
-    </joint>
-    <!-- END JOINTS -->
-    <!-- START Delete if not needed -->
-    <!-- Standard frames for industrial robots. Also useful for manipulators.
-         (ROS-I specs - https://wiki.ros.org/Industrial/Tutorials/WorkingWithRosIndustrialRobotSupportPackages#Standardised_links_.2F_frames)-->
-    <joint name="${prefix}base_link-base_joint" type="fixed">
-      <origin xyz="0 0 0" rpy="0 0 0"/>
-      <parent link="${prefix}base_link"/>
-      <child link="${prefix}base"/>
-    </joint>
-    <joint name="${prefix}tool0-flange_joint" type="fixed">
-      <origin xyz="0 0 0" rpy="0 0 0"/>
-      <parent link="${prefix}tool0"/>
-      <child link="${prefix}flange"/>
-    </joint>
-    <!-- END Delete if not needed  -->
   </xacro:macro>
 </robot>
