Commit message: Added ekf support and did some fixes to urdf

File: src/robot_description/urdf/robot_x/robot_x_macro.xacro (robot description, xacro)
@@ -8,5 +8,5 @@
       <!-- <xacro:default_inertial/> -->
       <visual>
-        <origin xyz="0 0 0" rpy="0 0 0"/>
+        <origin xyz="0.0065 0 0" rpy="0 0 0"/>
         <geometry>
           <cylinder length="0.05" radius="0.1675"/> <!-- robot radius 335mm -->
@@ -15,5 +15,5 @@
       </visual>
       <collision>
-        <origin xyz="0 0 0" rpy="0 0 0"/>
+        <origin xyz="0.0065 0 0" rpy="0 0 0"/>
         <geometry>
           <cylinder length="0.05" radius="0.1675"/>
@@ -55,7 +55,14 @@
       </collision>
     </link>
+    <link name="${prefix}imu_link"/>
+    <joint name="${prefix}imu_joint" type="fixed">
+        <parent link="${prefix}base_link"/>
+        <child link="${prefix}imu_link"/>
+        <origin xyz="0.04 0 0.03"
+                rpy="0 0 0"/>
+    </joint>
     <!-- Left wheel joint -->
     <joint name="${prefix}left_wheel_joint" type="continuous">
-      <origin xyz="-0.0065 0.1175 0" rpy="0 0 0"/> <!-- x behind center, y left -->
+      <origin xyz="0 0.1175 0" rpy="0 0 0"/> <!-- x behind center, y left -->
       <axis xyz="0 1 0"/> <!-- rotation around Y-axis -->
       <parent link="${prefix}base_link"/>
@@ -65,5 +72,5 @@
     <!-- Right wheel joint -->
     <joint name="${prefix}right_wheel_joint" type="continuous">
-      <origin xyz="-0.0065 -0.1175 0" rpy="0 0 0"/> <!-- x behind center, y right -->
+      <origin xyz="-0 -0.1175 0" rpy="0 0 0"/> <!-- x behind center, y right -->
       <axis xyz="0 1 0"/>
       <parent link="${prefix}base_link"/>
