Commit message: Add files via upload

File: src/robot_description/urdf/robot_x.urdf.xacro (robot description, xacro)
@@ -7,5 +7,6 @@
   <xacro:arg name="sim_gazebo_classic" default="false"/>
   <xacro:arg name="sim_gazebo" default="false"/>
-  <xacro:arg name="simulation_controllers" default=""/>
+  <xacro:arg name="simulation_controllers" default="" />
+  <xacro:arg name="wheelbase" default="0.235"/> <!-- set for your model -->
   <xacro:include filename="$(find robot_description)/urdf/robot_x/robot_x_macro.xacro"/>
   <xacro:include filename="$(find robot_description)/urdf/robot_x/robot_x_macro.ros2_control.xacro"/>
@@ -17,4 +18,5 @@
     <origin xyz="0 0 0" rpy="0 0 0"/>          <!-- position robot in the world -->
   </xacro:robot_x>
+  <!-- Load ros2_control macro with parameters -->
   <xacro:robot_x_ros2_control
     name="robot_x"
@@ -24,4 +26,5 @@
     sim_gazebo_classic="$(arg sim_gazebo_classic)"
     sim_gazebo="$(arg sim_gazebo)"
-    simulation_controllers="$(arg simulation_controllers)"/>
+    simulation_controllers="$(arg simulation_controllers)"
+    wheelbase="$(arg wheelbase)"/>
 </robot>

File: src/robot_description/urdf/robot_x/robot_x_macro.ros2_control.xacro (robot description, xacro)
@@ -8,5 +8,6 @@
                sim_gazebo_classic:=false
                sim_gazebo:=false
-               simulation_controllers"
+               simulation_controllers
+               wheelbase"
                >
     <ros2_control name="${name}" type="system">
@@ -25,29 +26,75 @@
           <plugin>robot_hardware_interface/RobotHardwareInterface</plugin>
         </xacro:unless>
+        <param name="wheelbase">${wheelbase}</param>
       </hardware>
+      <!-- Joint definitions -->
+      <joint name="${prefix}left_wheel_joint">
+        <command_interface name="velocity">
+          <param name="min">-301</param>
+          <param name="max">301</param>
+        </command_interface>
+        <state_interface name="position"/>
+      </joint>
+      <joint name="${prefix}right_wheel_joint">
+        <command_interface name="velocity">
+          <param name="min">-301</param>
+          <param name="max">301</param>
+        </command_interface>
+        <state_interface name="position"/>
+      </joint>
+      <joint name="${prefix}clean_mode_joint">
+        <command_interface name="velocity">
+          <param name="min">0</param>
+          <param name="max">7</param>
+        </command_interface>
+        <state_interface name="position"/>
+      </joint>
       <joint name="${prefix}linear_velocity_joint">
-        <command_interface name="velocity">     <!-- Add/Remove interfaces as needed -->
-          <param name="min">-200</param><!-- -1 -->
-          <param name="max">200</param><!-- 1 -->
+        <command_interface name="velocity">
+          <param name="min">-0.5</param>
+          <param name="max">0.5</param>
         </command_interface>
-        <command_interface name="position"/>
-        <state_interface name="position">
-          <param name="initial_value">0.0</param>
-        </state_interface>
-        <state_interface name="velocity"/>
-        <state_interface name="acceleration"/>
+        <state_interface name="position"/>
       </joint>
       <joint name="${prefix}angular_velocity_joint">
-        <command_interface name="velocity">     <!-- Add/Remove interfaces as needed -->
-          <param name="min">-200</param> <!-- -1 -->
-          <param name="max">200</param> <!-- 1 -->
+        <command_interface name="velocity">
+          <param name="min">-1.0</param>
+          <param name="max">1.0</param>
         </command_interface>
-        <command_interface name="position"/>
-        <state_interface name="position">
-          <param name="initial_value">0.0</param>
-        </state_interface>
-        <state_interface name="velocity"/>
-        <state_interface name="acceleration"/>
+        <state_interface name="position"/>
       </joint>
+      <!-- Joint definitions end -->
+      <!-- Sensor definitions -->
+      <sensor name="${prefix}sensor_data">
+        <state_interface name="bumps_right"/>
+        <state_interface name="bumps_left"/>
+        <state_interface name="wheeldrops_right"/>
+        <state_interface name="wheeldrops_left"/>
+        <state_interface name="wheeldrops_caster"/>
+        <state_interface name="wall"/>
+        <state_interface name="cliff_left"/>
+        <state_interface name="cliff_front_left"/>
+        <state_interface name="cliff_front_right"/>
+        <state_interface name="cliff_right"/>
+        <state_interface name="virtual_wall"/>
+        <state_interface name="motor_overcurrents_sidebrush"/>
+        <state_interface name="motor_overcurrents_vacuum"/>
+        <state_interface name="motor_overcurrents_mainbrush"/>
+        <state_interface name="motor_overcurrents_driveright"/>
+        <state_interface name="motor_overcurrents_driveleft"/>
+        <state_interface name="dirt_detector_left"/>
+        <state_interface name="dirt_detector_right"/>
+        <state_interface name="remote_opcode"/>
+        <state_interface name="button_max"/>
+        <state_interface name="button_clean"/>
+        <state_interface name="button_spot"/>
+        <state_interface name="button_power"/>
+        <state_interface name="charging_state"/>
+        <state_interface name="voltage"/>
+        <state_interface name="current"/>
+        <state_interface name="temperature"/>
+        <state_interface name="charge"/>
+        <state_interface name="capacity"/>
+      </sensor>
     </ros2_control>
     <xacro:if value="$(arg sim_gazebo_classic)">

File: src/robot_description/urdf/robot_x/robot_x_macro.xacro (robot description, xacro)
@@ -23,5 +23,5 @@
       </collision>
     </link>
-    <link name="${prefix}linear_velocity_link">
+    <link name="${prefix}left_wheel_link">
       <!-- Default inertial for Gazebo - copy and edit block from 'common.xacro'
       to get more realistic behavior -->
@@ -44,5 +44,5 @@
       </collision>
     </link>
-    <link name="${prefix}angular_velocity_link">
+    <link name="${prefix}right_wheel_link">
       <!-- Default inertial for Gazebo - copy and edit block from 'common.xacro'
            to get more realistic behavior-->
@@ -72,18 +72,18 @@
     </joint>
     <!-- joint 1 -->
-    <joint name="${prefix}linear_velocity_joint" type="revolute">
+    <joint name="${prefix}left_wheel_joint" type="revolute">
       <origin xyz="0 0 0.3" rpy="${pi} 0 0"/>
       <axis xyz="0 0 1"/>
       <limit effort="0" lower="${radians(-180)}" upper="${radians(180)}" velocity="${radians(180)}"/>
       <parent link="${prefix}base_link"/>  <!-- Specify parent link -->
-      <child link="${prefix}linear_velocity_link"/>  <!-- Specify child link -->
+      <child link="${prefix}left_wheel_link"/>  <!-- Specify child link -->
     </joint>
     <!-- joint 2 -->
-    <joint name="${prefix}angular_velocity_joint" type="revolute">
+    <joint name="${prefix}right_wheel_joint" type="revolute">
       <origin xyz="0 0 -0.3" rpy="${pi/2} 0 0"/>
       <axis xyz="0 0 1"/>
       <limit effort="0" lower="${radians(-180)}" upper="${radians(180)}" velocity="${radians(180)}"/>
-      <parent link="${prefix}linear_velocity_link"/>  <!-- Specify parent link -->
-      <child link="${prefix}angular_velocity_link"/>  <!-- Specify child link -->
+      <parent link="${prefix}base_link"/>  <!-- Specify parent link -->
+      <child link="${prefix}right_wheel_link"/>  <!-- Specify child link -->
     </joint>
   </xacro:macro>

Commit message: Full rework

File: src/robot_description/urdf/robot_x.urdf.xacro (robot description, xacro)
@@ -12,9 +12,11 @@
   <xacro:include filename="$(find robot_description)/urdf/robot_x/robot_x_macro.ros2_control.xacro"/>
   <!-- create link fixed to the "world" -->
-  <link name="world"/>
+  <!-- <link name="world"/> -->
   <!-- Load robot's macro with parameters -->
   <!-- set prefix if multiple robots are used -->
-  <xacro:robot_x prefix="$(arg prefix)" parent="world">
-    <origin xyz="0 0 0" rpy="0 0 0"/>          <!-- position robot in the world -->
+  <!-- <xacro:robot_x prefix="$(arg prefix)" parent="world">
+    <origin xyz="0 0 0" rpy="0 0 0"/>
+  </xacro:robot_x> -->
+  <xacro:robot_x prefix="$(arg prefix)">
   </xacro:robot_x>
   <!-- Load ros2_control macro with parameters -->

File: src/robot_description/urdf/robot_x/robot_x_macro.ros2_control.xacro (robot description, xacro)
@@ -43,72 +43,89 @@
         <state_interface name="position"/>
       </joint>
-      <joint name="${prefix}clean_mode_joint">
-        <command_interface name="velocity">
-          <param name="min">0</param>
-          <param name="max">7</param>
-        </command_interface>
-        <state_interface name="position"/>
-      </joint>
-      <joint name="${prefix}linear_velocity_joint">
-        <command_interface name="velocity">
-          <param name="min">-0.5</param>
-          <param name="max">0.5</param>
-        </command_interface>
-        <state_interface name="position"/>
-      </joint>
-      <joint name="${prefix}angular_velocity_joint">
-        <command_interface name="velocity">
-          <param name="min">-1.0</param>
-          <param name="max">1.0</param>
-        </command_interface>
-        <state_interface name="position"/>
-      </joint>
       <!-- Joint definitions end -->
       <!-- Sensor definitions -->
       <sensor name="${prefix}sensor_data">
-        <state_interface name="bumps_right"/>
-        <state_interface name="bumps_left"/>
-        <state_interface name="wheeldrops_right"/>
-        <state_interface name="wheeldrops_left"/>
-        <state_interface name="wheeldrops_caster"/>
-        <state_interface name="wall"/>
-        <state_interface name="cliff_left"/>
-        <state_interface name="cliff_front_left"/>
-        <state_interface name="cliff_front_right"/>
-        <state_interface name="cliff_right"/>
-        <state_interface name="virtual_wall"/>
-        <state_interface name="motor_overcurrents_sidebrush"/>
-        <state_interface name="motor_overcurrents_vacuum"/>
-        <state_interface name="motor_overcurrents_mainbrush"/>
-        <state_interface name="motor_overcurrents_driveright"/>
-        <state_interface name="motor_overcurrents_driveleft"/>
-        <state_interface name="dirt_detector_left"/>
-        <state_interface name="dirt_detector_right"/>
-        <state_interface name="remote_opcode"/>
-        <state_interface name="button_max"/>
-        <state_interface name="button_clean"/>
-        <state_interface name="button_spot"/>
-        <state_interface name="button_power"/>
-        <state_interface name="charging_state"/>
-        <state_interface name="voltage"/>
-        <state_interface name="current"/>
-        <state_interface name="temperature"/>
-        <state_interface name="charge"/>
-        <state_interface name="capacity"/>
+        <state_interface name="bumps_right"/>                  <!-- hw_sensor_states[0] -->
+        <state_interface name="bumps_left"/>                   <!-- hw_sensor_states[1] -->
+        <state_interface name="wheeldrops_right"/>             <!-- hw_sensor_states[2] -->
+        <state_interface name="wheeldrops_left"/>              <!-- hw_sensor_states[3] -->
+        <state_interface name="wall"/>                         <!-- hw_sensor_states[4] -->
+        <state_interface name="cliff_left"/>                   <!-- hw_sensor_states[5] -->
+        <state_interface name="cliff_front_left"/>            <!-- hw_sensor_states[6] -->
+        <state_interface name="cliff_front_right"/>            <!-- hw_sensor_states[7] -->
+        <state_interface name="cliff_right"/>                  <!-- hw_sensor_states[8] -->
+        <state_interface name="virtual_wall"/>                 <!-- hw_sensor_states[9] -->
+        <state_interface name="motor_overcurrents_sidebrush"/> <!-- hw_sensor_states[10] -->
+        <state_interface name="motor_overcurrents_vacuum"/>    <!-- hw_sensor_states[11] -->
+        <state_interface name="motor_overcurrents_mainbrush"/> <!-- hw_sensor_states[12] -->
+        <state_interface name="motor_overcurrents_driveright"/> <!-- hw_sensor_states[13] -->
+        <state_interface name="motor_overcurrents_driveleft"/> <!-- hw_sensor_states[14] -->
+        <state_interface name="dirt_detect"/>                  <!-- hw_sensor_states[15] -->
+        <state_interface name="remote_opcode"/>                <!-- hw_sensor_states[16] -->
+        <state_interface name="button_clean"/>                 <!-- hw_sensor_states[17] -->
+        <state_interface name="button_spot"/>                  <!-- hw_sensor_states[18] -->
+        <state_interface name="button_dock"/>                  <!-- hw_sensor_states[19] -->
+        <state_interface name="button_minute"/>                <!-- hw_sensor_states[20] -->
+        <state_interface name="button_hour"/>                  <!-- hw_sensor_states[21] -->
+        <state_interface name="button_day"/>                   <!-- hw_sensor_states[22] -->
+        <state_interface name="button_schedule"/>              <!-- hw_sensor_states[23] -->
+        <state_interface name="button_clock"/>                 <!-- hw_sensor_states[24] -->
+        <state_interface name="distance"/>                     <!-- hw_sensor_states[25] -->
+        <state_interface name="angle"/>                        <!-- hw_sensor_states[26] -->
+        <state_interface name="charging_state"/>               <!-- hw_sensor_states[27] -->
+        <state_interface name="voltage"/>                      <!-- hw_sensor_states[28] -->
+        <state_interface name="current"/>                      <!-- hw_sensor_states[29] -->
+        <state_interface name="temperature"/>                  <!-- hw_sensor_states[30] -->
+        <state_interface name="charge"/>                       <!-- hw_sensor_states[31] -->
+        <state_interface name="capacity"/>                     <!-- hw_sensor_states[32] -->
+        <state_interface name="wall_signal"/>                  <!-- hw_sensor_states[33] -->
+        <state_interface name="cliff_left_signal"/>            <!-- hw_sensor_states[34] -->
+        <state_interface name="cliff_front_left_signal"/>      <!-- hw_sensor_states[35] -->
+        <state_interface name="cliff_front_right_signal"/>     <!-- hw_sensor_states[36] -->
+        <state_interface name="cliff_right_signal"/>           <!-- hw_sensor_states[37] -->
+        <state_interface name="charger_available"/>            <!-- hw_sensor_states[38] -->
+        <state_interface name="open_interface_mode"/>          <!-- hw_sensor_states[39] -->
+        <state_interface name="song_number"/>                  <!-- hw_sensor_states[40] -->
+        <state_interface name="song_playing"/>                 <!-- hw_sensor_states[41] -->
+        <state_interface name="oi_stream_num_packets"/>        <!-- hw_sensor_states[42] -->
+        <state_interface name="velocity"/>                     <!-- hw_sensor_states[43] -->
+        <state_interface name="radius"/>                      <!-- hw_sensor_states[44] -->
+        <state_interface name="velocity_right"/>               <!-- hw_sensor_states[45] -->
+        <state_interface name="velocity_left"/>                <!-- hw_sensor_states[46] -->
+        <state_interface name="encoder_counts_left"/>          <!-- hw_sensor_states[47] -->
+        <state_interface name="encoder_counts_right"/>         <!-- hw_sensor_states[48] -->
+        <state_interface name="light_bumper"/>                 <!-- hw_sensor_states[49] -->
+        <state_interface name="light_bump_left"/>              <!-- hw_sensor_states[50] -->
+        <state_interface name="light_bump_front_left"/>        <!-- hw_sensor_states[51] -->
+        <state_interface name="light_bump_center_left"/>       <!-- hw_sensor_states[52] -->
+        <state_interface name="light_bump_center_right"/>     <!-- hw_sensor_states[53] -->
+        <state_interface name="light_bump_front_right"/>      <!-- hw_sensor_states[54] -->
+        <state_interface name="light_bump_right"/>            <!-- hw_sensor_states[55] -->
+        <state_interface name="ir_opcode_left"/>              <!-- hw_sensor_states[56] -->
+        <state_interface name="ir_opcode_right"/>             <!-- hw_sensor_states[57] -->
+        <state_interface name="left_motor_current"/>           <!-- hw_sensor_states[58] -->
+        <state_interface name="right_motor_current"/>         <!-- hw_sensor_states[59] -->
+        <state_interface name="main_brush_current"/>          <!-- hw_sensor_states[60] -->
+        <state_interface name="side_brush_current"/>          <!-- hw_sensor_states[61] -->
+        <state_interface name="stasis"/>                      <!-- hw_sensor_states[62] -->
+        <state_interface name="x"/>                         <!-- hw_sensor_states[63] -->
+        <state_interface name="y"/>                         <!-- hw_sensor_states[64] -->
+        <state_interface name="theta"/>                     <!-- hw_sensor_states[65] -->
       </sensor>
-      <!-- Side brush -->
+      <gpio name="${prefix}main_brush">
+        <command_interface name="duty_cycle"/>
+        <state_interface name="duty_cycle"/>
+      </gpio>
       <gpio name="${prefix}side_brush">
-        <state_interface name="state"/>
-        <command_interface name="state"/>
+        <command_interface name="duty_cycle"/>
+        <state_interface name="duty_cycle"/>
       </gpio>
-      <!-- Vacuum -->
       <gpio name="${prefix}vacuum">
-        <command_interface name="state"/>
-        <state_interface name="state"/>
+        <command_interface name="duty_cycle"/>
+        <state_interface name="duty_cycle"/>
       </gpio>
-      <!-- Main brush -->
-      <gpio name="${prefix}motors">
-        <command_interface name="state"/>
-        <state_interface name="state"/>
+      <gpio name="${prefix}mode">
+        <command_interface name="value"/>
+        <state_interface name="value"/>
       </gpio>
     </ros2_control>

File: src/robot_description/urdf/robot_x/robot_x_macro.xacro (robot description, xacro)
@@ -3,13 +3,12 @@
   <xacro:include filename="$(find robot_description)/urdf/common/inertials.xacro"/>
   <xacro:include filename="$(find robot_description)/urdf/common/materials.xacro"/>
-  <xacro:macro name="robot_x" params="prefix parent *origin">
+  <xacro:macro name="robot_x" params="prefix">
+    <!-- BASE LINK -->
     <link name="${prefix}base_link">
-      <!-- Add geometry or inertia properties -->
       <xacro:default_inertial/>
       <visual>
         <origin xyz="0 0 0" rpy="0 0 0"/>
         <geometry>
-          <cylinder length="0.3" radius="0.3"/>
-          <!--           <mesh filename="package://robot_description/meshes/robot_x/visual/base_link.dae" /> -->
+          <cylinder length="0.05" radius="0.1675"/> <!-- robot radius 335mm -->
         </geometry>
         <material name="black"/>
@@ -18,18 +17,15 @@
         <origin xyz="0 0 0" rpy="0 0 0"/>
         <geometry>
-          <cylinder length="0.3" radius="0.3"/>
-          <!--           <mesh filename="package://robot_description/meshes/robot_x/collision/base_link.stl" /> -->
+          <cylinder length="0.05" radius="0.1675"/>
         </geometry>
       </collision>
     </link>
+    <!-- LEFT WHEEL LINK -->
     <link name="${prefix}left_wheel_link">
-      <!-- Default inertial for Gazebo - copy and edit block from 'common.xacro'
-      to get more realistic behavior -->
       <xacro:default_inertial/>
       <visual>
         <origin xyz="0 0 0" rpy="0 0 0"/>
         <geometry>
-          <cylinder length="0.3" radius="0.15"/>
-          <!--           <mesh filename="package://robot_description/meshes/robot_x/visual/link1.dae" /> -->
+          <cylinder length="0.015" radius="0.036"/> <!-- wheel thickness 15mm, radius 36mm -->
         </geometry>
         <material name="blue"/>
@@ -38,19 +34,15 @@
         <origin xyz="0 0 0" rpy="0 0 0"/>
         <geometry>
-          <cylinder length="0.3" radius="0.15"/>
-          <!--           <mesh filename="package://robot_description/meshes/robot_x/collision/link1.stl" /> -->
+          <cylinder length="0.015" radius="0.036"/>
         </geometry>
-        <material name="green"/>
       </collision>
     </link>
+    <!-- RIGHT WHEEL LINK -->
     <link name="${prefix}right_wheel_link">
-      <!-- Default inertial for Gazebo - copy and edit block from 'common.xacro'
-           to get more realistic behavior-->
       <xacro:default_inertial/>
       <visual>
         <origin xyz="0 0 0" rpy="0 0 0"/>
         <geometry>
-          <cylinder length="0.3" radius="0.15"/>
-          <!--           <mesh filename="package://robot_description/meshes/robot_x/visual/link2.dae" /> -->
+          <cylinder length="0.015" radius="0.036"/>
         </geometry>
         <material name="grey"/>
@@ -59,31 +51,23 @@
         <origin xyz="0 0 0" rpy="0 0 0"/>
         <geometry>
-          <cylinder length="0.3" radius="0.15"/>
-          <!--           <mesh filename="package://robot_description/meshes/robot_x/collision/link2.stl"  /> -->
+          <cylinder length="0.015" radius="0.036"/>
         </geometry>
       </collision>
     </link>
-    <!-- JOINTS -->
-    <!-- base_joint fixes base_link to the environment -->
-    <joint name="${prefix}base_joint" type="fixed">
-      <xacro:insert_block name="origin"/>
-      <parent link="${parent}"/>
-      <child link="${prefix}base_link"/>
+    <!-- Left wheel joint -->
+    <joint name="${prefix}left_wheel_joint" type="continuous">
+      <origin xyz="-0.0065 0.1175 0" rpy="0 0 0"/> <!-- x behind center, y left -->
+      <axis xyz="0 1 0"/> <!-- rotation around Y-axis -->
+      <parent link="${prefix}base_link"/>
+      <child link="${prefix}left_wheel_link"/>
+      <limit effort="10" velocity="300"/>
     </joint>
-    <!-- joint 1 -->
-    <joint name="${prefix}left_wheel_joint" type="revolute">
-      <origin xyz="0 0 0.3" rpy="${pi} 0 0"/>
-      <axis xyz="0 0 1"/>
-      <limit effort="0" lower="${radians(-180)}" upper="${radians(180)}" velocity="${radians(180)}"/>
-      <parent link="${prefix}base_link"/>  <!-- Specify parent link -->
-      <child link="${prefix}left_wheel_link"/>  <!-- Specify child link -->
-    </joint>
-    <!-- joint 2 -->
-    <joint name="${prefix}right_wheel_joint" type="revolute">
-      <origin xyz="0 0 -0.3" rpy="${pi/2} 0 0"/>
-      <axis xyz="0 0 1"/>
-      <limit effort="0" lower="${radians(-180)}" upper="${radians(180)}" velocity="${radians(180)}"/>
-      <parent link="${prefix}base_link"/>  <!-- Specify parent link -->
-      <child link="${prefix}right_wheel_link"/>  <!-- Specify child link -->
+    <!-- Right wheel joint -->
+    <joint name="${prefix}right_wheel_joint" type="continuous">
+      <origin xyz="-0.0065 -0.1175 0" rpy="0 0 0"/> <!-- x behind center, y right -->
+      <axis xyz="0 1 0"/>
+      <parent link="${prefix}base_link"/>
+      <child link="${prefix}right_wheel_link"/>
+      <limit effort="10" velocity="300"/>
     </joint>
   </xacro:macro>
